Commit message: Steren bot URDF added for kinematics activity

File: class_ws/src/motor_sim/urdf/steren.urdf (robot description, URDF)
Before this commit: robot steren, 5 links, 4 joints
Links:
- link link1: geometry visual cylinder length=0.05 radius=0.05
- link link2: geometry visual cylinder length=0.05 radius=0.05
- link link3: geometry visual cylinder length=0.05 radius=0.05
- link link4: geometry visual cylinder length=0.05 radius=0.05
